File: hardware/kicad/pca9306.kicad_sch (KiCad schematic)
At the start: 8 parts, among them J2 Omron, U4 PCA9306D, U4C1 100P

Commit message: keep on working the schematics and PCB
Changed lines of the file:
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@@
 		(on_board yes)
 		(dnp no)
-		(fields_autoplaced yes)
 		(property "Reference" "#PWR027"
 			(at 153.67 76.2 0)
@@
 		)
 		(property "Value" "+5V"
-			(at 160.655 76.1999 90)
+			(at 156.21 78.105 90)
 			(effects
 				(font
@@
 		(on_board yes)
 		(dnp no)
-		(fields_autoplaced yes)
 		(property "Reference" "#PWR028"
 			(at 109.22 87.63 0)
@@
 		)
 		(property "Value" "+3V3"
-			(at 109.22 78.74 0)
+			(at 109.22 80.01 0)
 			(effects
 				(font
@@
 		(on_board yes)
 		(dnp no)
-		(fields_autoplaced yes)
 		(property "Reference" "#PWR024"
 			(at 97.79 97.79 0)
@@
 		)
 		(property "Value" "+3V3"
-			(at 90.17 97.7899 90)
+			(at 95.885 95.885 90)
 			(effects
 				(font
@@
 		(on_board yes)
 		(dnp no)
-		(fields_autoplaced yes)
 		(property "Reference" "#PWR025"
 			(at 123.19 82.55 0)
@@
 		)
 		(property "Value" "GND"
-			(at 123.19 81.28 0)
+			(at 123.19 80.01 0)
 			(effects
 				(font
@@
 		)
 		(property "Value" "+5V"
-			(at 157.48 99.06 90)
+			(at 158.75 98.425 90)
 			(effects
 				(font
@@
 		)
 		(property "Value" "100P"
-			(at 130.81 82.55 90)
-			(effects
-				(font
+			(at 130.81 81.915 90)
+			(effects
+				(font
