File: hardware/kicad/pcb_nixie.kicad_pcb (KiCad board)
At the start: 6 copper layers, 90.7 x 90.7 mm, 44 parts, among them J1 MCU-SWD, J2 Omron, J3 GPS-M8N, J4 Power-supply, J5 Littelfuse-0218.020HXP, J6 OLED, U1 STM32L4A6RGTx, U1C1 4.7U, U1C2 100N, U1C3 100N, U1C4 100N, U1C5 100N, U1C6 100N, U1C7 100N, U2 TXB0104PW, U2C1 100N, U2C2 100N, U3 K155id1, U3C1 1U, U4 PCA9306D, U4C1 100P

Commit message: keep on working the schematics and PCB
Parts:
- moved U3 87.4 mm to (61.7, 105.6)
- moved U3C1 87.4 mm to (60.7, 112.3)
- moved R1 12.1 mm to (129.1, 116.9)
- moved R5 10.8 mm to (153.3, 81.3)
- moved R4 9.80 mm to (136.1, 122.3)
- moved R3 7.85 mm to (173.6, 107.2)
- moved R9 5.77 mm to (133.8, 105.6)
- moved R7 5.11 mm to (173.9, 90.8)
- moved U2 4.55 mm to (155.0, 121.0)
- moved U2C2 4.55 mm to (157.6, 117.9)
- moved U2C1 4.55 mm to (152.3, 117.9)
- moved NX1 3.66 mm to (152.3, 105.9)
Changed lines of the file:
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@@
 	(footprint "Package_DIP:SMDIP-16_W7.62mm"
 		(layer "F.Cu")
-		(at 148.975816 101.894544 90)
+		(at 61.654503 105.639461 90)
 		(descr "16-lead surface-mounted (SMD) DIP package, row spacing 7.62mm (300 mils)")
 		(tags "SMD DIP DIL PDIP SMDIP 2.54mm 7.62mm 300mil")
@@
 	(footprint "Nixie:nixie_socket_manual"
 		(layer "F.Cu")
-		(at 148.917916 107.368266)
+		(at 152.254522 105.852781)
 		(property "Reference" "NX1"
 			(at -6.689618 -5.969043 0)
@@
 	(footprint "Resistor_SMD:R_1206_3216Metric"
 		(layer "F.Cu")
-		(at 138.755816 108.589706 180)
+		(at 133.819062 105.594543 180)
 		(descr "Resistor SMD 1206 (3216 Metric), square (rectangular) end terminal, IPC-7351 nominal, (Body size source: IPC-SM-782 page 72, https://www.pcb-3d.com/wordpress/wp-content/uploads/ipc-sm-782a_amendment_1_and_2.pdf), generated with kicad-footprint-generator")
 		(tags "resistor")
@@
 	(footprint "Package_SO:TSSOP-14_4.4x5mm_P0.65mm"
 		(layer "F.Cu")
-		(at 151.672916 117.851917)
+		(at 154.997639 120.964948)
 		(descr "TSSOP, 14 Pin (JEDEC MO-153 Var AB-1 https://www.jedec.org/document_search?search_api_views_fulltext=MO-153), generated with kicad-footprint-generator ipc_gullwing_generator.py")
 		(tags "TSSOP SO")
@@
 	(footprint "Resistor_SMD:R_1206_3216Metric"
 		(layer "F.Cu")
-		(at 169.600959 93.529477 90)
+		(at 173.942197 90.840214 90)
 		(descr "Resistor SMD 1206 (3216 Metric), square (rectangular) end terminal, IPC-7351 nominal, (Body size source: IPC-SM-782 page 72, https://www.pcb-3d.com/wordpress/wp-content/uploads/ipc-sm-782a_amendment_1_and_2.pdf), generated with kicad-footprint-generator")
 		(tags "resistor")
@@
 	(footprint "Resistor_SMD:R_1206_3216Metric"
 		(layer "F.Cu")
-		(at 139.8088 113.195433 -90)
+		(at 136.085666 122.264871 -90)
 		(descr "Resistor SMD 1206 (3216 Metric), square (rectangular) end terminal, IPC-7351 nominal, (Body size source: IPC-SM-782 page 72, https://www.pcb-3d.com/wordpress/wp-content/uploads/ipc-sm-782a_amendment_1_and_2.pdf), generated with kicad-footprint-generator")
 		(tags "resistor")
@@
 	(footprint "Resistor_SMD:R_1206_3216Metric"
 		(layer "F.Cu")
-		(at 152.08478 92.026688 90)
+		(at 153.338771 81.287021 90)
 		(descr "Resistor SMD 1206 (3216 Metric), square (rectangular) end terminal, IPC-7351 nominal, (Body size source: IPC-SM-782 page 72, https://www.pcb-3d.com/wordpress/wp-content/uploads/ipc-sm-782a_amendment_1_and_2.pdf), generated with kicad-footprint-generator")
 		(tags "resistor")
@@
 	(footprint "Resistor_SMD:R_1206_3216Metric"
 		(layer "F.Cu")
-		(at 166.794034 103.191774 90)
+		(at 173.568759 107.16519 90)
 		(descr "Resistor SMD 1206 (3216 Metric), square (rectangular) end terminal, IPC-7351 nominal, (Body size source: IPC-SM-782 page 72, https://www.pcb-3d.com/wordpress/wp-content/uploads/ipc-sm-782a_amendment_1_and_2.pdf), generated with kicad-footprint-generator")
 		(tags "resistor")
@@
 		)
 		(fp_text user "${REFERENCE}"
-			(at 0 0 90)
+			(at -0.727064 0.91 90)
 			(layer "F.Fab")
 			(effects
@@
 	(footprint "Resistor_SMD:R_1206_3216Metric"
 		(layer "F.Cu")
-		(at 140.7188 113.7318 -90)
+		(at 129.073361 116.856729 -90)
 		(descr "Resistor SMD 1206 (3216 Metric), square (rectangular) end terminal, IPC-7351 nominal, (Body size source: IPC-SM-782 page 72, https://www.pcb-3d.com/wordpress/wp-content/uploads/ipc-sm-782a_amendment_1_and_2.pdf), generated with kicad-footprint-generator")
 		(tags "resistor")
@@
 		)
 		(fp_text user "${REFERENCE}"
-			(at 0 0 90)
+			(at 0 5.058122 90)
 			(layer "F.Fab")
 			(effects
@@
 	(footprint "Capacitor_SMD:C_0603_1608Metric"
 		(layer "B.Cu")
-		(at 149.012916 114.805434 180)
+		(at 152.337639 117.918465 180)
 		(descr "Capacitor SMD 0603 (1608 Metric), square (rectangular) end terminal, IPC-7351 nominal, (Body size source: IPC-SM-782 page 76, https://www.pcb-3d.com/wordpress/wp-content/uploads/ipc-sm-782a_amendment_1_and_2.pdf), generated with kicad-footprint-generator")
 		(tags "capacitor")
@@
 	(footprint "Capacitor_SMD:C_0603_1608Metric"
 		(layer "B.Cu")
-		(at 154.295541 114.750028 180)
+		(at 157.620264 117.863059 180)
 		(descr "Capacitor SMD 0603 (1608 Metric), square (rectangular) end terminal, IPC-7351 nominal, (Body size source: IPC-SM-782 page 76, https://www.pcb-3d.com/wordpress/wp-content/uploads/ipc-sm-782a_amendment_1_and_2.pdf), generated with kicad-footprint-generator")
 		(tags "capacitor")
@@
 	(footprint "Resistor_SMD:R_0603_1608Metric"
 		(layer "B.Cu")
-		(at 147.971521 108.533596 180)
+		(at 60.650208 112.278513 180)
 		(descr "Resistor SMD 0603 (1608 Metric), square (rectangular) end terminal, IPC-7351 nominal, (Body size source: IPC-SM-782 page 72, https://www.pcb-3d.com/wordpress/wp-content/uploads/ipc-sm-782a_amendment_1_and_2.pdf), generated with kicad-footprint-generator")
 		(tags "resistor")
@@
 	)
 	(gr_line
-		(start 156.025667 115.898703)
-		(end 156.025667 114.970939)
+		(start 159.35039 119.011734)
+		(end 159.35039 118.08397)
 		(stroke
 			(width 0.2)
@@
 	)
 	(gr_line
-		(start 148.233347 115.901917)
-		(end 147.207315 115.901917)
+		(start 151.55807 119.014948)
+		(end 150.532038 119.014948)
 		(stroke
 			(width 0.2)
@@
 	)
 	(gr_line
-		(start 155.166186 115.895734)
-		(end 156.025667 115.898703)
+		(start 158.490909 119.008765)
+		(end 159.35039 119.011734)
 		(stroke
 			(width 0.2)
@@
 	)
 	(gr_line
-		(start 147.207315 115.901917)
-		(end 147.207315 115.018441)
+		(start 150.532038 119.014948)
+		(end 150.532038 118.131472)
 		(stroke
 			(width 0.2)
@@
 	)
 	(via blind
-		(at 149.668632 108.374412)
+		(at 62.347319 112.119329)
 		(size 0.3)
 		(drill 0.25)
@@
 	)
 	(via blind
-		(at 147.222078 114.842371)
+		(at 150.546801 117.955402)
 		(size 0.3)
 		(drill 0.25)
@@
 	)
 	(via blind
-		(at 156.013118 114.768497)
+		(at 159.337841 117.881528)
 		(size 0.3)
 		(drill 0.25)
@@
 	)
 	(via blind
-		(at 150.753664 108.365543)
+		(at 63.432351 112.11046)
 		(size 0.3)
 		(drill 0.25)
@@
 	)
 	(via blind
-		(at 146.248802 108.351201)
+		(at 58.927489 112.096118)
 		(size 0.3)
 		(drill 0.250012)
@@
 	)
 	(via blind
-		(at 152.51703 114.761933)
+		(at 155.841753 117.874964)
 		(size 0.3)
 		(drill 0.25)
@@
 	)
 	(via blind
-		(at 150.798426 114.749108)
+		(at 154.123149 117.862139)
 		(size 0.3)
 		(drill 0.25)
@@
 	)
 	(group ""
-		(members "199c9d7d-1017-4719-8a87-dec201b08eca" "22eddda6-d3be-4592-add2-23a61478cced")
-	)
-	(group ""
